Commit message: updated zed package, fixed TF issue

File: zed-ros2-wrapper/zed_wrapper/urdf/zed_macro.urdf.xacro (robot description, xacro)
@@ -76,9 +76,9 @@
       </collision>
     </link>
-    <joint name="${name}_camera_center_joint" type="fixed">
+    <!--joint name="${name}_camera_center_joint" type="fixed">
       <parent link="${name}_base_link"/>
       <child link="${name}_camera_center"/>
       <origin xyz="0 0 ${height/2}" rpy="0 ${bottom_slope} 0" />
-    </joint>
+    </joint-->
     <!-- Left Camera -->
     <link name="${name}_left_camera_frame" />
